File: ARG2026_Beacon_circuit.kicad_sch (KiCad schematic)
At the start: 21 parts, among them J1 Conn_01x02_Pin, J2 Conn_01x02_Pin, Q1 IRLML0030, U1 CH32V002A4M6

Commit message: Test_push
Other:
- note added: "hello"
Changed lines of the file:
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@@
 	(generator_version "10.0")
 	(paper "A4")
+	(text "hello\n"
+		(exclude_from_sim no)
+		(at 100.076 105.41 0)
+		(effects
+			(font
+				(size 1.27 1.27)
+			)
+		)
+	)
 	(junction
 		(at 116.84 90.17)

Commit message: 既に適応済みの部品を流用
Parts:
- added D7: LED, LED_THT:LED_D3.0mm, symbol Device:LED
- added R9: 1k, Resistor_THT:R_Axial_DIN0207_L6.3mm_D2.5mm_P10.16mm_Horizontal, symbol Device:R
- added SW1: SW_SPDT, Button_Switch_THT:SW_Slide-03_Wuerth-WS-SLTV_10x2.5x6.4_P2.54mm, symbol Switch:SW_SPDT
Connections:
- net GND: now also D7.1 (K)
- net VDD: now also R9.1, SW1.2 (B); no longer BT1.1 (+)
- new net: D7.2 (A), R9.2
- new net: BT1.1 (+), SW1.1 (A)
- no-connect marks 12 -> 13

Commit message: シルクスクリーンに値を追加、チェック
Parts:
- R1, R2, R3, R4, R5, R6: value 5R1 -> 6R8
Changed lines of the file:
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@@
 			)
 		)
-		(property "Value" "5R1"
+		(property "Value" "6R8"
 			(at 123.19 60.706 90)
 			(show_name no)
@@
 			)
 		)
-		(property "Value" "5R1"
+		(property "Value" "6R8"
 			(at 123.19 78.486 90)
 			(show_name no)
@@
 			)
 		)
-		(property "Value" "5R1"
+		(property "Value" "6R8"
 			(at 123.19 69.596 90)
 			(show_name no)
@@
 			)
 		)
-		(property "Value" "5R1"
+		(property "Value" "6R8"
 			(at 123.19 96.266 90)
 			(show_name no)
@@
 			)
 		)
-		(property "Value" "5R1"
+		(property "Value" "6R8"
 			(at 123.19 51.816 90)
 			(show_name no)
@@
 			)
 		)
-		(property "Value" "5R1"
+		(property "Value" "6R8"
 			(at 123.19 87.376 90)
 			(show_name no)

Commit message: improve silkscreen of PCB
Parts:
- C1: value 470 -> 470u
Changed lines of the file:
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@@
 			)
 		)
-		(property "Value" "470"
+		(property "Value" "470u"
 			(at 104.14 79.1209 0)
 			(show_name no)
