File: ARG2026_Beacon_circuit.kicad_pcb (KiCad board)
At the start: 2 copper layers, 100 x 86.6 mm, 31 parts, among them J1 Conn_01x02_Pin, J2 Conn_01x02_Pin, Q1 IRLML0030, SW1 SW_SPDT, U1 CH32V002A4M6

Commit message: Fix DRC_Error
Parts:
- removed ?: , clipboard:8ea2c0b2-452e-4bc2-b55e-ed6b78fbe1c2
Changed lines of the file:
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@@
 		(embedded_fonts no)
 	)
-	(footprint "clipboard:8ea2c0b2-452e-4bc2-b55e-ed6b78fbe1c2"
-		(layer "F.Cu")
-		(at 199.238267 97.55 180)
-		(property "Reference" ""
-			(at 0 0 0)
-			(layer "F.SilkS")
-			(effects
-				(font
-					(size 1.27 1.27)
-				)
-			)
-		)
-		(property "Value" ""
-			(at 0 0 0)
-			(layer "F.Fab")
-			(effects
-				(font
-					(size 1.27 1.27)
-				)
-			)
-		)
-		(property "Datasheet" ""
-			(at 0 0 0)
-			(layer "F.Fab")
-			(hide yes)
-			(effects
-				(font
-					(size 1.27 1.27)
-				)
-			)
-		)
-		(property "Description" ""
-			(at 0 0 0)
-			(layer "F.Fab")
-			(hide yes)
-			(effects
-				(font
-					(size 1.27 1.27)
-				)
-			)
-		)
-		(duplicate_pad_numbers_are_jumpers no)
-		(fp_line
-			(start 0 0)
-			(end 0 0.448267)
-			(stroke
-				(width 0.070576)
-				(type default)
-			)
-			(layer "F.SilkS")
-		)
-		(fp_line
-			(start 0 0)
-			(end 0 -0.448267)
-			(stroke
-				(width 0.070576)
-				(type default)
-			)
-			(layer "F.SilkS")
-		)
-		(fp_line
-			(start 0 0)
-			(end -0.448329 0)
-			(stroke
-				(width 0.070576)
-				(type default)
-			)
-			(layer "F.SilkS")
-		)
-		(fp_line
-			(start -0.448329 0)
-			(end -0.896622 0)
-			(stroke
-				(width 0.070576)
-				(type default)
-			)
-			(layer "F.SilkS")
-		)
-		(fp_line
-			(start -0.896622 0)
-			(end 1.793156 0)
-			(stroke
-				(width 0.070576)
-				(type default)
-			)
-			(layer "F.SilkS")
-		)
-		(fp_poly
-			(pts
-				(xy 0.881653 0.448038) (xy 0.896534 -0.448267) (xy 0 0)
-			)
-			(stroke
-				(width 0.070576)
-				(type solid)
-			)
-			(fill yes)
-			(layer "F.SilkS")
-		)
-		(embedded_fonts no)
-	)
 	(footprint "MountingHole:MountingHole_3.2mm_M3"
 		(layer "F.Cu")
@@
 		(sheetname "/")
 		(sheetfile "ARG2026_Beacon_circuit.kicad_sch")
-		(units
-			(unit
-				(name "A")
-				(pins "1" "2")
-			)
-		)
 		(attr through_hole)
 		(duplicate_pad_numbers_are_jumpers no)
 		(fp_line
+			(start 1 -3)
+			(end 1 -2.551733)
+			(stroke
+				(width 0.070576)
+				(type default)
+			)
+			(layer "F.SilkS")
+		)
+		(fp_line
+			(start 1 -3)
+			(end 1 -3.448267)
+			(stroke
+				(width 0.070576)
+				(type default)
+			)
+			(layer "F.SilkS")
+		)
+		(fp_line
+			(start 1 -3)
+			(end 0.551671 -3)
+			(stroke
+				(width 0.070576)
+				(type default)
+			)
+			(layer "F.SilkS")
+		)
+		(fp_line
+			(start 0.551671 -3)
+			(end 0.103378 -3)
+			(stroke
+				(width 0.070576)
+				(type default)
+			)
+			(layer "F.SilkS")
+		)
+		(fp_line
+			(start 0.103378 -3)
+			(end 2.793156 -3)
+			(stroke
+				(width 0.070576)
+				(type default)
+			)
+			(layer "F.SilkS")
+		)
+		(fp_line
 			(start -0.29 1.08)
 			(end -0.29 1.236)
@@
 			(layer "F.SilkS")
 		)
+		(fp_poly
+			(pts
+				(xy 1.881653 -2.551962) (xy 1.896534 -3.448267) (xy 1 -3)
+			)
+			(stroke
+				(width 0.070576)
+				(type solid)
+			)
+			(fill yes)
+			(layer "F.SilkS")
+		)

Commit message: GND塗りつぶしを忘れてました
Routing:
- added copper zone on F.Cu, net GND
Changed lines of the file:
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@@
+	)
+	(zone
+		(net "GND")
+		(layer "F.Cu")
+		(hatch edge 0.5)
+		(connect_pads
+			(clearance 0.5)
+		)
+		(min_thickness 0.25)
+		(fill yes
+			(thermal_gap 0.5)
+			(thermal_bridge_width 0.5)
+			(island_removal_mode 0)
+		)
+		(polygon
+			(pts
+				(xy 196.07 57.81) (xy 246.05 57.81) (xy 271.07 101.13) (xy 246.07 144.42) (xy 196.07 144.41) (xy 171.06 101.098086)
+			)
+		)
 	)
 	(zone
